File: effects-switcher.kicad_pcb (KiCad board)
At the start: 2 copper layers, 257 x 41 mm, 57 parts, among them J12 Conn_01x02, J34 Conn_01x02, J4 Conn_01x02, J56 Conn_01x02, Q1 2N3904, Q2 2N3904, Q3 2N3904, Q4 2N3904, Q5 2N3904, Q6 2N3904, U1 LM7805

Commit message: revised silk screen
Parts:
- renumbered L1-In1 to L1-In, L1-Out1 to L1-Out, L2-In1 to L2-In, L2-Out1 to L2-Out, L3-In1 to L3-In, L3-Out1 to L3-Out, L4-In1 to L4-In, L4-Out1 to L4-Out
Changed lines of the file:
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@@
     (property "Sheetname" "")
     (attr through_hole)
-    (fp_text reference "L2-In1" (at 6.35 8.1 90) (layer "F.SilkS")
+    (fp_text reference "L2-In" (at 6.35 8.1 90) (layer "F.SilkS")
       (effects (font (size 1 1) (thickness 0.15)))
     )
@@
     (property "Sheetname" "")
     (attr through_hole)
-    (fp_text reference "L2-Out1" (at 6.35 8.1 90) (layer "F.SilkS")
+    (fp_text reference "L2-Out" (at 6.35 8.1 90) (layer "F.SilkS")
       (effects (font (size 1 1) (thickness 0.15)))
     )
@@
     (property "Sheetname" "")
     (attr through_hole)
-    (fp_text reference "L1-In1" (at 6.35 8.1 90) (layer "F.SilkS")
+    (fp_text reference "L1-In" (at 6.35 8.1 90) (layer "F.SilkS")
       (effects (font (size 1 1) (thickness 0.15)))
     )
@@
     (property "Sheetname" "")
     (attr through_hole)
-    (fp_text reference "L1-Out1" (at 6.35 8.1 90) (layer "F.SilkS")
+    (fp_text reference "L1-Out" (at 6.35 8.1 90) (layer "F.SilkS")
       (effects (font (size 1 1) (thickness 0.15)))
     )
@@
     (property "Sheetname" "")
     (attr through_hole)
-    (fp_text reference "L3-Out1" (at 6.35 8.1 90) (layer "F.SilkS")
+    (fp_text reference "L3-Out" (at 6.35 8.1 90) (layer "F.SilkS")
       (effects (font (size 1 1) (thickness 0.15)))
     )
@@
     (property "Sheetname" "")
     (attr through_hole)
-    (fp_text reference "L4-In1" (at 6.35 8.1 90) (layer "F.SilkS")
+    (fp_text reference "L4-In" (at 6.35 8.1 90) (layer "F.SilkS")
       (effects (font (size 1 1) (thickness 0.15)))
     )
@@
     (property "Sheetname" "")
     (attr through_hole)
-    (fp_text reference "L4-Out1" (at 6.35 8.1 90) (layer "F.SilkS")
+    (fp_text reference "L4-Out" (at 6.35 8.1 90) (layer "F.SilkS")
       (effects (font (size 1 1) (thickness 0.15)))
     )
@@
     (property "Sheetname" "")
     (attr through_hole)
-    (fp_text reference "L3-In1" (at 6.35 8.1 90) (layer "F.SilkS")
-      (effects (font (size 1 1) (thickness 0.15)))
-    )
+    (fp_text reference "L3-In" (at 6.35 8.1 90) (layer "F.SilkS")
+      (effects (font (size 1 1) (thickness 0.15)))
+    )

Commit message: removed 9v out
Parts:
- removed JDC2: Barrel_Jack_Switch, Connector_BarrelJack:BarrelJack_Horizontal
- J1: renamed from In; value AudioJack3_SwitchSTR -> In
- J10: renamed from L4-In; value AudioJack3_SwitchSTR -> L4-In
- J11: renamed from L4-Out; value AudioJack3_SwitchSTR -> L4-Out
- J2: renamed from Out; value AudioJack3_SwitchSTR -> Out
- J3: renamed from Tuner; value AudioJack3_SwitchSTR -> Tuner
- J4: renamed from L1-In; value AudioJack3_SwitchSTR -> L1-In
- J5: renamed from L1-Out; value AudioJack3_SwitchSTR -> L1-Out
- J6: renamed from L2-In; value AudioJack3_SwitchSTR -> L2-In
- J7: renamed from L2-Out; value AudioJack3_SwitchSTR -> L2-Out
- J8: renamed from L3-In; value AudioJack3_SwitchSTR -> L3-In
- J9: renamed from L3-Out; value AudioJack3_SwitchSTR -> L3-Out
- K1: renamed from Bypass; value EC2-4.5NU -> Bypass; footprint Relay_THT:Relay_DPDT_Kemet_EC2 -> Nate:Relay_DPDT_Kemet_EC2
- K2: renamed from Tuner; value EC2-4.5NU -> Tuner; footprint Relay_THT:Relay_DPDT_Kemet_EC2 -> Nate:Relay_DPDT_Kemet_EC2
- K3: renamed from Loop1; value EC2-4.5NU -> Loop1; footprint Relay_THT:Relay_DPDT_Kemet_EC2 -> Nate:Relay_DPDT_Kemet_EC2
- K4: renamed from Loop2; value EC2-4.5NU -> Loop2; footprint Relay_THT:Relay_DPDT_Kemet_EC2 -> Nate:Relay_DPDT_Kemet_EC2
- K5: renamed from Loop3; value EC2-4.5NU -> Loop3; footprint Relay_THT:Relay_DPDT_Kemet_EC2 -> Nate:Relay_DPDT_Kemet_EC2
- K6: renamed from Loop4; value EC2-4.5NU -> Loop4; footprint Relay_THT:Relay_DPDT_Kemet_EC2 -> Nate:Relay_DPDT_Kemet_EC2
- U1: value LM7805 -> 7805
- moved C2 8.62 mm to (239.5, 27.4)
- moved U1 8.01 mm to (245.1, 19.9)
- moved C1 5.21 mm to (238.4, 19.8)
- moved J+9 1.99 mm to (241.0, 14.0)
- renumbered J4 to J+5, JDC1 to J+9
Routing:
- net +9V: track 1.70 -> 0.00 mm
Other:
- board size 257 x 41 mm -> 249 x 41 mm
- board text removed: "9V Out"

Commit message: Revert "removed 9v out"
This reverts commit 68eda4370ce2c703412f077e884cf7a60c7e0849.
Parts:
- added JDC2: Barrel_Jack_Switch, Connector_BarrelJack:BarrelJack_Horizontal, F.Cu at (251.0, 14.0)
- Bypass: renamed from K1; value Bypass -> EC2-4.5NU; footprint Nate:Relay_DPDT_Kemet_EC2 -> Relay_THT:Relay_DPDT_Kemet_EC2
- In: renamed from J1; value In -> AudioJack3_SwitchSTR
- L1-In: renamed from J4; value L1-In -> AudioJack3_SwitchSTR
- L1-Out: renamed from J5; value L1-Out -> AudioJack3_SwitchSTR
- L2-In: renamed from J6; value L2-In -> AudioJack3_SwitchSTR
- L2-Out: renamed from J7; value L2-Out -> AudioJack3_SwitchSTR
- L3-In: renamed from J8; value L3-In -> AudioJack3_SwitchSTR
- L3-Out: renamed from J9; value L3-Out -> AudioJack3_SwitchSTR
- L4-In: renamed from J10; value L4-In -> AudioJack3_SwitchSTR
- L4-Out: renamed from J11; value L4-Out -> AudioJack3_SwitchSTR
- Loop1: renamed from K3; value Loop1 -> EC2-4.5NU; footprint Nate:Relay_DPDT_Kemet_EC2 -> Relay_THT:Relay_DPDT_Kemet_EC2
- Loop2: renamed from K4; value Loop2 -> EC2-4.5NU; footprint Nate:Relay_DPDT_Kemet_EC2 -> Relay_THT:Relay_DPDT_Kemet_EC2
- Loop3: renamed from K5; value Loop3 -> EC2-4.5NU; footprint Nate:Relay_DPDT_Kemet_EC2 -> Relay_THT:Relay_DPDT_Kemet_EC2
- Loop4: renamed from K6; value Loop4 -> EC2-4.5NU; footprint Nate:Relay_DPDT_Kemet_EC2 -> Relay_THT:Relay_DPDT_Kemet_EC2
- Out: renamed from J2; value Out -> AudioJack3_SwitchSTR
- Tuner: renamed from J3; value Tuner -> AudioJack3_SwitchSTR
- Tuner: renamed from K2; value Tuner -> EC2-4.5NU; footprint Nate:Relay_DPDT_Kemet_EC2 -> Relay_THT:Relay_DPDT_Kemet_EC2
- U1: value 7805 -> LM7805
- moved C2 8.62 mm to (248.0, 26.0)
- moved U1 8.01 mm to (253.1, 20.5)
- moved C1 5.21 mm to (243.5, 19.0)
- moved JDC1 1.99 mm to (239.0, 14.0)
- renumbered J+5 to J4, J+9 to JDC1
Routing:
- net +9V: track 0.00 -> 1.70 mm
Other:
- board size 249 x 41 mm -> 257 x 41 mm
- board text added: "9V Out"
